File: pihat_template/hardware/Ideal_Diode.sch (KiCad schematic (older format))
At the start: 4 parts, among them Q1 BSS138, U5 DMMT5401

Commit message: added farnell part no.
Parts:
- Q1: Farnell Part No. (none) -> 9845330
- R11: Farnell Part No. (none) -> 2324717
- R12: Farnell Part No. (none) -> 6379860
- U5: Farnell Part No. (none) -> 1773583
Changed lines of the file:
@@
 LIBS:xilinx
 LIBS:Zilog
+LIBS:cat24c32hu4i-gt3
+LIBS:DMMT5401
+LIBS:fdc5614p
+LIBS:lm1117
+LIBS:lm3489
+LIBS:max1164x
+LIBS:mcp23017
+LIBS:raspberry_pi_+_conn
 LIBS:pihat_template-cache
 EELAYER 25 0
@@
 F 3 "" H 6000 3100 60  0000 C CNN
 F 4 "621-DMG2305UX-13" H 6000 3100 60  0001 C CNN "Mouser Part No."
+F 5 "9845330" H 6000 3100 60  0001 C CNN "Farnell Part No."
 	1    6000 3100
 	0    -1   -1   0
@@
 F 3 "" H 5850 3700 47  0000 C CNN
 F 4 "621-DMMT5401-7-F" H 6000 4000 60  0001 C CNN "Mouser Part No."
+F 5 "1773583" H 6000 4000 60  0001 C CNN "Farnell Part No."
 	1    6000 4000
 	1    0    0    -1
@@
 F 3 "" H 6200 4800 30  0000 C CNN
 F 4 "667-ERJ-2RKF4702X" V 6200 4800 60  0001 C CNN "Mouser Part No."
+F 5 "6379860" V 6200 4800 60  0001 C CNN "Farnell Part No."
 	1    6200 4800
 	1    0    0    -1
@@
 F 3 "" H 5800 4800 30  0000 C CNN
 F 4 "71-CRCW0402-10K-E3" V 5800 4800 60  0001 C CNN "Mouser Part No."
+F 5 "2324717" V 5800 4800 60  0001 C CNN "Farnell Part No."
 	1    5800 4800
 	1    0    0    -1

Commit message: added  and links to 3D models for modules in project lib
Parts:
- Q1: footprint w_smd_trans:sot23 -> project:sot23
- R11, R12: footprint w_smd_resistors:r_0402 -> project:r_0402
- U5: footprint w_smd_trans:sot23-6 -> project:sot23-6
Changed lines of the file:
@@
 F 0 "Q1" H 6000 2951 40  0000 R CNN
 F 1 "BSS138" H 6000 3250 40  0000 R CNN
-F 2 "w_smd_trans:sot23" H 5870 3202 29  0000 C CNN
+F 2 "project:sot23" H 5870 3202 29  0000 C CNN
 F 3 "" H 6000 3100 60  0000 C CNN
 F 4 "621-DMG2305UX-13" H 6000 3100 60  0001 C CNN "Mouser Part No."
@@
 F 0 "U5" H 5700 4150 47  0000 C CNN
 F 1 "DMMT5401" H 6450 3800 47  0000 C CNN
-F 2 "w_smd_trans:sot23-6" H 5850 3700 47  0001 C CNN
+F 2 "project:sot23-6" H 5850 3700 47  0001 C CNN
 F 3 "" H 5850 3700 47  0000 C CNN
 F 4 "621-DMMT5401-7-F" H 6000 4000 60  0001 C CNN "Mouser Part No."
@@
 F 0 "R12" V 6280 4800 50  0000 C CNN
 F 1 "47k" V 6207 4801 50  0000 C CNN
-F 2 "w_smd_resistors:r_0402" V 6130 4800 30  0001 C CNN
+F 2 "project:r_0402" V 6130 4800 30  0001 C CNN
 F 3 "" H 6200 4800 30  0000 C CNN
 F 4 "667-ERJ-2RKF4702X" V 6200 4800 60  0001 C CNN "Mouser Part No."
@@
 F 0 "R11" V 5880 4800 50  0000 C CNN
 F 1 "10k" V 5807 4801 50  0000 C CNN
-F 2 "w_smd_resistors:r_0402" V 5730 4800 30  0001 C CNN
+F 2 "project:r_0402" V 5730 4800 30  0001 C CNN
 F 3 "" H 5800 4800 30  0000 C CNN
 F 4 "71-CRCW0402-10K-E3" V 5800 4800 60  0001 C CNN "Mouser Part No."

Commit message: refactor large components
Parts:
- R11, R12: footprint project:r_0402 -> project:r_0805
Changed lines of the file:
@@
 F 0 "R12" V 6280 4800 50  0000 C CNN
 F 1 "47k" V 6207 4801 50  0000 C CNN
-F 2 "project:r_0402" V 6130 4800 30  0001 C CNN
+F 2 "project:r_0805" V 6130 4800 30  0001 C CNN
 F 3 "" H 6200 4800 30  0000 C CNN
 F 4 "667-ERJ-2RKF4702X" V 6200 4800 60  0001 C CNN "Mouser Part No."
@@
 F 0 "R11" V 5880 4800 50  0000 C CNN
 F 1 "10k" V 5807 4801 50  0000 C CNN
-F 2 "project:r_0402" V 5730 4800 30  0001 C CNN
+F 2 "project:r_0805" V 5730 4800 30  0001 C CNN
 F 3 "" H 5800 4800 30  0000 C CNN
 F 4 "71-CRCW0402-10K-E3" V 5800 4800 60  0001 C CNN "Mouser Part No."
