File: pihat_template/hardware/pihat_template.sch (KiCad schematic (older format))
At the start: 29 parts, among them P1 CONN_01X02, P2 CONN_01X02, P3 Raspberry_Pi_+_Conn, U1 LM3489, U2 CAT24C32HU4I-GT3, U3 FDC5614P, U4 LM1117IMPX-ADJ

Commit message: update components
Parts:
- D1: Farnell Part No. (none) -> 2628293; Mouser Part No. 512-MBRS140 -> (none)
- U1: footprint w_smd_dil:msoic-8 -> project:VSSOP-8_3.0x3.0mm_Pitch0.65mm; Farnell Part No. (none) -> 1312570; Mouser Part No. 926-LM3489MM/NOPB -> (none)
Changed lines of the file:
@@
 F 0 "U1" H 2450 9050 60  0000 C CNN
 F 1 "LM3489" H 3350 8400 60  0000 C CNN
-F 2 "w_smd_dil:msoic-8" H 2850 9000 60  0001 C CNN
+F 2 "project:VSSOP-8_3.0x3.0mm_Pitch0.65mm" H 2850 9000 60  0001 C CNN
 F 3 "" H 2850 9000 60  0000 C CNN
-F 4 "926-LM3489MM/NOPB" H 2850 9000 60  0001 C CNN "Mouser Part No."
+F 4 "1312570" H 2850 9000 60  0001 C CNN "Farnell Part No."
 	1    2850 9000
 	1    0    0    -1
@@
 F 2 "w_smd_diode:do214aa" H 4200 8700 60  0001 C CNN
 F 3 "" H 4200 8700 60  0000 C CNN
-F 4 "512-MBRS140" H 4200 8700 60  0001 C CNN "Mouser Part No."
+F 4 "2628293" H 4200 8700 60  0001 C CNN "Farnell Part No."
 	1    4200 8700
 	0    -1   -1   0

Commit message: added farnell part no.
Parts:
- C1: Farnell Part No. (none) -> 1973367
- C2, C4, C5, C7: Farnell Part No. (none) -> 2210822
- C3: Farnell Part No. (none) -> 1907278
- C6: Farnell Part No. (none) -> 2466348
- C8: Farnell Part No. (none) -> 2346885
- D3: Farnell Part No. (none) -> 1652083
- JP1, P1: Farnell Part No. (none) -> ?
- L1: Farnell Part No. (none) -> 2061671
- P2: Farnell Part No. (none) -> 2008004
- P3: Farnell Part No. (none) -> 2668422
- R1: Farnell Part No. (none) -> 2324716
- R10: Farnell Part No. (none) -> 2379848
- R2: Farnell Part No. (none) -> 2379837
- R3, R5: Farnell Part No. (none) -> 2563570
- R4: Farnell Part No. (none) -> 2324732
- R6: Farnell Part No. (none) -> 2379844
- R7: Farnell Part No. (none) -> 2324717
- R8: Farnell Part No. (none) -> 2379851
- R9: Farnell Part No. (none) -> 2379835
- U2: Farnell Part No. (none) -> 2463727
- U3: Farnell Part No. (none) -> 1471036
- U4: Farnell Part No. (none) -> 2463930
Changed lines of the file:
@@
 LIBS:xilinx
 LIBS:Zilog
+LIBS:cat24c32hu4i-gt3
+LIBS:DMMT5401
+LIBS:fdc5614p
+LIBS:lm1117
+LIBS:lm3489
+LIBS:max1164x
+LIBS:mcp23017
+LIBS:raspberry_pi_+_conn
 LIBS:pihat_template-cache
 EELAYER 25 0
@@
 F 3 "" H 5750 3900 60  0000 C CNN
 F 4 "517-30340-6002" H 5750 3900 60  0001 C CNN "Mouser Part No."
+F 5 "2668422" H 5750 3900 60  0001 C CNN "Farnell Part No."
 	1    5750 3900
 	-1   0    0    -1
@@
 F 3 "" H 3000 4400 60  0000 C CNN
 F 4 "698-CAT24C32YI-GT3" H 3000 4400 60  0001 C CNN "Mouser Part No."
+F 5 "2463727" H 3000 4400 60  0001 C CNN "Farnell Part No."
 	1    3000 4400
 	1    0    0    -1
@@
 F 3 "" H 2000 4650 30  0000 C CNN
 F 4 "754-RR0510P-102D" V 2000 4650 60  0001 C CNN "Mouser Part No."
+F 5 "2324716" V 2000 4650 60  0001 C CNN "Farnell Part No."
 	1    2000 4650
 	1    0    0    -1
@@
 F 2 "w_pin_strip:pin_strip_2" H 950 5000 60  0001 C CNN
 F 3 "" H 950 5000 60  0000 C CNN
+F 4 "?" H 950 5000 60  0001 C CNN "Farnell Part No."
 	1    950  5000
 	-1   0    0    1
@@
 F 3 "" H 3850 4000 30  0000 C CNN
 F 4 "71-CRCW04023K90FKED" V 3850 4000 60  0001 C CNN "Mouser Part No."
+F 5 "2563570" V 3850 4000 60  0001 C CNN "Farnell Part No."
 	1    3850 4000
 	1    0    0    -1
@@
 F 3 "" H 4100 4000 30  0000 C CNN
 F 4 "71-CRCW04023K90FKED" V 4100 4000 60  0001 C CNN "Mouser Part No."
+F 5 "2563570" V 4100 4000 60  0001 C CNN "Farnell Part No."
 	1    4100 4000
 	1    0    0    -1
@@
 F 2 "w_smd_resistors:r_0603" H 1600 5200 60  0001 C CNN
 F 3 "" H 1600 5200 60  0000 C CNN
+F 4 "?" H 1600 5200 60  0001 C CNN "Farnell Part No."
 	1    1600 5200
 	1    0    0    1
@@
 F 3 "" H 2000 8700 30  0000 C CNN
 F 4 "71-CRCW0402-24K-E3" V 2000 8700 60  0001 C CNN "Mouser Part No."
+F 5 "2379837" V 2000 8700 60  0001 C CNN "Farnell Part No."
 	1    2000 8700
 	1    0    0    -1
@@
 F 3 "" H 1550 9550 60  0000 C CNN
 F 4 "810-C1005X5R1H104K" H 1550 9550 60  0001 C CNN "Mouser Part No."
+F 5 "2210822" H 1550 9550 60  0001 C CNN "Farnell Part No."
 	1    1550 9550
 	1    0    0    -1
@@
 F 3 "" H 1100 8650 300 0000 C CNN
 F 4 "647-UUR1H470MCL6GS" H 1100 8650 60  0001 C CNN "Mouser Part No."
+F 5 "1973367" H 1100 8650 60  0001 C CNN "Farnell Part No."
 	1    1100 8650
 	1    0    0    -1
@@
 F 3 "" H 1800 8700 60  0000 C CNN
 F 4 "810-C1005C0G2A102J5C" H 1800 8700 60  0001 C CNN "Mouser Part No."
+F 5 "1907278" H 1800 8700 60  0001 C CNN "Farnell Part No."
 	1    1800 8700
 	1    0    0    -1
@@
 F 3 "" H 3900 8700 30  0000 C CNN
 F 4 "667-ERJ-P6WJ271V" V 3900 8700 60  0001 C CNN "Mouser Part No."
+F 5 "2324732" V 3900 8700 60  0001 C CNN "Farnell Part No."
 	1    3900 8700
 	1    0    0    -1
@@
 F 3 "" H 4600 8200 60  0000 C CNN
 F 4 "652-SRN8040-220M" V 4600 8200 60  0001 C CNN "Mouser Part No."
+F 5 "2061671" V 4600 8200 60  0001 C CNN "Farnell Part No."
 	1    4600 8200
 	0    -1   -1   0
@@
 F 3 "" H 5050 8700 30  0000 C CNN
 F 4 "594-MCT06030C3002FP5" V 5050 8700 60  0001 C CNN "Mouser Part No."
+F 5 "2379844" V 5050 8700 60  0001 C CNN "Farnell Part No."
 	1    5050 8700
 	1    0    0    -1
@@
 F 3 "" H 5050 9650 30  0000 C CNN
 F 4 "71-CRCW0603-10K-E3" V 5050 9650 60  0001 C CNN "Mouser Part No."
+F 5 "2324717" V 5050 9650 60  0001 C CNN "Farnell Part No."
 	1    5050 9650
 	1    0    0    -1
@@
 F 3 "" H 3100 8500 60  0000 C CNN
 F 4 "512-FDC5614P" H 3250 8350 60  0001 C CNN "Mouser Part No."
+F 5 "1471036" H 3250 8350 60  0001 C CNN "Farnell Part No."
 	1    3250 8350
 	-1   0    0    -1
@@
 F 3 "" H 8100 8250 60  0000 C CNN
 F 4 "926-M1117IMPXADJNOPB" H 8100 8300 60  0001 C CNN "Mouser Part No."
+F 5 "2463930" H 8100 8300 60  0001 C CNN "Farnell Part No."
 	1    8100 8300
 	1    0    0    -1
@@
 F 3 "" H 7350 8650 300 0000 C CNN
 F 4 "5985-AVS16V100-F" H 7350 8650 60  0001 C CNN "Mouser Part No."
+F 5 "2466348" H 7350 8650 60  0001 C CNN "Farnell Part No."
 	1    7350 8650
 	1    0    0    -1
@@
 F 3 "" H 8100 9300 30  0000 C CNN
 F 4 "594-MCT06030C3900FP5" V 8100 9300 60  0001 C CNN "Mouser Part No."
+F 5 "2379851" V 8100 9300 60  0001 C CNN "Farnell Part No."
 	1    8100 9300
 	1    0    0    -1
@@
 F 3 "" H 9150 8600 30  0000 C CNN
 F 4 "754-RR0816P-241D" V 9150 8600 60  0001 C CNN "Mouser Part No."
+F 5 "2379835" V 9150 8600 60  0001 C CNN "Farnell Part No."
 	1    9150 8600
 	1    0    0    -1
@@
 F 3 "" H 10550 8550 60  0000 C CNN
 F 4 "743-HT-191USD" H 10550 8550 60  0001 C CNN "Mouser Part No."
+F 5 "1652083" H 10550 8550 60  0001 C CNN "Farnell Part No."
 	1    10550 8550
 	0    1    1    0
@@
 F 3 "" H 10550 9200 30  0000 C CNN
 F 4 "71-CRCW0603316RFKEB" V 10550 9200 60  0001 C CNN "Mouser Part No."
+F 5 "2379848" V 10550 9200 60  0001 C CNN "Farnell Part No."
 	1    10550 9200
 	1    0    0    -1
@@
 F 3 "" H 4800 8700 60  0000 C CNN
 F 4 "810-C1005X5R1H104K" H 4800 8700 60  0001 C CNN "Mouser Part No."
+F 5 "2210822" H 4800 8700 60  0001 C CNN "Farnell Part No."
 	1    4800 8700
 	1    0    0    -1
@@
 F 3 "" H 9500 8550 60  0000 C CNN
 F 4 "810-C1005X5R1H104K" H 9500 8550 60  0001 C CNN "Mouser Part No."
+F 5 "2210822" H 9500 8550 60  0001 C CNN "Farnell Part No."
 	1    9500 8550
 	1    0    0    -1
@@
 F 3 "" H 3350 6950 60  0000 C CNN
 F 4 "651-1904383" H 3350 6950 60  0001 C CNN "Mouser Part No."
+F 5 "2008004" H 3350 6950 60  0001 C CNN "Farnell Part No."
 	1    3350 6950
 	1    0    0    -1
@@
 F 3 "" H 2350 4700 60  0000 C CNN
 F 4 "810-C1005X5R1H104K" H 2350 4700 60  0001 C CNN "Mouser Part No."
+F 5 "2210822" H 2350 4700 60  0001 C CNN "Farnell Part No."
 	1    2350 4700
 	1    0    0    -1
@@
 F 3 "" H 9900 8550 60  0000 C CNN
 F 4 "810-C1005X5R1H104K" H 9900 8550 60  0001 C CNN "Mouser Part No."
+F 5 "2346885" H 9900 8550 60  0001 C CNN "Farnell Part No."
 	1    9900 8550
 	1    0    0    -1

Commit message: added  and links to 3D models for modules in project lib
Parts:
- C1: footprint w_smd_cap:c_elec_6.3x7.7 -> project:c_elec_6.3x7.7
- C2, C3, C4, C5, C7, C8: footprint w_smd_cap:c_0402 -> project:c_0402
- C6: footprint w_smd_cap:c_elec_4x5.3 -> project:c_elec_4x5.3
- D1: footprint w_smd_diode:do214aa -> project:do214aa
- D3: footprint w_smd_leds:Led_0603 -> project:Led_0603
- JP1: footprint w_smd_resistors:r_0603 -> project:r_0603
- L1: footprint w_smd_inductors:inductor_smd_8x5mm -> project:inductor_smd_8x5mm
- P1: footprint w_pin_strip:pin_strip_2 -> project:pin_strip_2
- P2: footprint w_conn_mkds:mkds_1,5-2 -> project:mkds_1,5-2
- P3: footprint w_conn_strip:vasch_strip_20x2 -> project:pin_socket_20x2
- R1, R10, R2, R3, R4, R5, R6, R7, R8, R9: footprint w_smd_resistors:r_0402 -> project:r_0402
- U2: footprint w_smd_dil:tssop-8 -> project:tssop-8
- U3: footprint w_smd_trans:sot23-6 -> project:sot23-6
- U4: footprint w_smd_trans:sot223 -> project:sot223
Changed lines of the file:
@@
 F 0 "P3" H 4650 5850 60  0000 C CNN
 F 1 "Raspberry_Pi_+_Conn" H 6050 2450 60  0000 C CNN
-F 2 "w_conn_strip:vasch_strip_20x2" H 5750 3900 60  0001 C CNN
+F 2 "project:pin_socket_20x2" H 5750 3900 60  0001 C CNN
 F 3 "" H 5750 3900 60  0000 C CNN
 F 4 "517-30340-6002" H 5750 3900 60  0001 C CNN "Mouser Part No."
@@
 F 0 "U2" H 2900 4550 60  0000 C CNN
 F 1 "CAT24C32HU4I-GT3" H 3400 3600 60  0000 C CNN
-F 2 "w_smd_dil:tssop-8" H 3000 4400 60  0001 C CNN
+F 2 "project:tssop-8" H 3000 4400 60  0001 C CNN
 F 3 "" H 3000 4400 60  0000 C CNN
 F 4 "698-CAT24C32YI-GT3" H 3000 4400 60  0001 C CNN "Mouser Part No."
@@
 F 0 "R1" V 2080 4650 40  0000 C CNN
 F 1 "1k" V 2007 4651 40  0000 C CNN
-F 2 "w_smd_resistors:r_0402" V 1930 4650 30  0001 C CNN
+F 2 "project:r_0402" V 1930 4650 30  0001 C CNN
 F 3 "" H 2000 4650 30  0000 C CNN
 F 4 "754-RR0510P-102D" V 2000 4650 60  0001 C CNN "Mouser Part No."
@@
 F 0 "P1" H 950 5150 50  0000 C CNN
 F 1 "CONN_01X02" V 1050 5000 50  0000 C CNN
-F 2 "w_pin_strip:pin_strip_2" H 950 5000 60  0001 C CNN
+F 2 "project:pin_strip_2" H 950 5000 60  0001 C CNN
 F 3 "" H 950 5000 60  0000 C CNN
 F 4 "?" H 950 5000 60  0001 C CNN "Farnell Part No."
@@
 F 0 "R3" V 3930 4000 40  0000 C CNN
 F 1 "3.9k" V 3857 4001 40  0000 C CNN
-F 2 "w_smd_resistors:r_0402" V 3780 4000 30  0001 C CNN
+F 2 "project:r_0402" V 3780 4000 30  0001 C CNN
 F 3 "" H 3850 4000 30  0000 C CNN
 F 4 "71-CRCW04023K90FKED" V 3850 4000 60  0001 C CNN "Mouser Part No."
@@
 F 0 "R5" V 4180 4000 40  0000 C CNN
 F 1 "3.9k" V 4107 4001 40  0000 C CNN
-F 2 "w_smd_resistors:r_0402" V 4030 4000 30  0001 C CNN
+F 2 "project:r_0402" V 4030 4000 30  0001 C CNN
 F 3 "" H 4100 4000 30  0000 C CNN
 F 4 "71-CRCW04023K90FKED" V 4100 4000 60  0001 C CNN "Mouser Part No."
@@
 F 0 "JP1" H 1600 5350 60  0000 C CNN
 F 1 "JUMPER" H 1600 5120 40  0000 C CNN
-F 2 "w_smd_resistors:r_0603" H 1600 5200 60  0001 C CNN
+F 2 "project:r_0603" H 1600 5200 60  0001 C CNN
 F 3 "" H 1600 5200 60  0000 C CNN
 F 4 "?" H 1600 5200 60  0001 C CNN "Farnell Part No."
@@
 F 0 "R2" V 2080 8700 40  0000 C CNN
 F 1 "24k" V 2007 8701 40  0000 C CNN
-F 2 "w_smd_resistors:r_0402" V 1930 8700 30  0001 C CNN
+F 2 "project:r_0402" V 1930 8700 30  0001 C CNN
 F 3 "" H 2000 8700 30  0000 C CNN
 F 4 "71-CRCW0402-24K-E3" V 2000 8700 60  0001 C CNN "Mouser Part No."
@@
 F 0 "C2" H 1550 9650 40  0000 L CNN
 F 1 "0.1uf" H 1556 9465 40  0000 L CNN
-F 2 "w_smd_cap:c_0402" H 1588 9400 30  0001 C CNN
+F 2 "project:c_0402" H 1588 9400 30  0001 C CNN
 F 3 "" H 1550 9550 60  0000 C CNN
 F 4 "810-C1005X5R1H104K" H 1550 9550 60  0001 C CNN "Mouser Part No."
@@
 F 0 "C1" H 1150 8750 40  0000 L CNN
 F 1 "50uf/50v" H 1150 8550 40  0000 L CNN
-F 2 "w_smd_cap:c_elec_6.3x7.7" H 1200 8500 30  0001 C CNN
+F 2 "project:c_elec_6.3x7.7" H 1200 8500 30  0001 C CNN
 F 3 "" H 1100 8650 300 0000 C CNN
 F 4 "647-UUR1H470MCL6GS" H 1100 8650 60  0001 C CNN "Mouser Part No."
@@
 F 0 "C3" H 1800 8800 40  0000 L CNN
 F 1 "1nf" H 1806 8615 40  0000 L CNN
-F 2 "w_smd_cap:c_0402" H 1838 8550 30  0001 C CNN
+F 2 "project:c_0402" H 1838 8550 30  0001 C CNN
 F 3 "" H 1800 8700 60  0000 C CNN
 F 4 "810-C1005C0G2A102J5C" H 1800 8700 60  0001 C CNN "Mouser Part No."
@@
 F 0 "R4" V 3980 8700 40  0000 C CNN
 F 1 "270" V 3907 8701 40  0000 C CNN
-F 2 "w_smd_resistors:r_0402" V 3830 8700 30  0001 C CNN
+F 2 "project:r_0402" V 3830 8700 30  0001 C CNN
 F 3 "" H 3900 8700 30  0000 C CNN
 F 4 "667-ERJ-P6WJ271V" V 3900 8700 60  0001 C CNN "Mouser Part No."
@@
 F 0 "D1" H 4200 8800 40  0000 C CNN
 F 1 "DIODESCH" H 4200 8600 40  0000 C CNN
-F 2 "w_smd_diode:do214aa" H 4200 8700 60  0001 C CNN
+F 2 "project:do214aa" H 4200 8700 60  0001 C CNN
 F 3 "" H 4200 8700 60  0000 C CNN
 F 4 "2628293" H 4200 8700 60  0001 C CNN "Farnell Part No."
@@
 F 0 "L1" V 4550 8200 40  0000 C CNN
 F 1 "22uH" V 4700 8200 40  0000 C CNN
-F 2 "w_smd_inductors:inductor_smd_8x5mm" H 4600 8200 60  0001 C CNN
+F 2 "project:inductor_smd_8x5mm" H 4600 8200 60  0001 C CNN
 F 3 "" H 4600 8200 60  0000 C CNN
 F 4 "652-SRN8040-220M" V 4600 8200 60  0001 C CNN "Mouser Part No."
@@
 F 0 "R6" V 5130 8700 40  0000 C CNN
 F 1 "30k" V 5057 8701 40  0000 C CNN
-F 2 "w_smd_resistors:r_0402" V 4980 8700 30  0001 C CNN
+F 2 "project:r_0402" V 4980 8700 30  0001 C CNN
 F 3 "" H 5050 8700 30  0000 C CNN
 F 4 "594-MCT06030C3002FP5" V 5050 8700 60  0001 C CNN "Mouser Part No."
@@
 F 0 "R7" V 5130 9650 40  0000 C CNN
 F 1 "10k" V 5057 9651 40  0000 C CNN
-F 2 "w_smd_resistors:r_0402" V 4980 9650 30  0001 C CNN
+F 2 "project:r_0402" V 4980 9650 30  0001 C CNN
 F 3 "" H 5050 9650 30  0000 C CNN
 F 4 "71-CRCW0603-10K-E3" V 5050 9650 60  0001 C CNN "Mouser Part No."
@@
 F 0 "U3" H 3100 8600 60  0000 C CNN
 F 1 "FDC5614P" H 3250 8100 60  0000 C CNN
-F 2 "w_smd_trans:sot23-6" H 3100 8500 60  0001 C CNN
+F 2 "project:sot23-6" H 3100 8500 60  0001 C CNN
 F 3 "" H 3100 8500 60  0000 C CNN
 F 4 "512-FDC5614P" H 3250 8350 60  0001 C CNN "Mouser Part No."
@@
 F 0 "U4" H 7850 8600 60  0000 C CNN
 F 1 "LM1117IMPX-ADJ" H 8550 8000 60  0000 C CNN
-F 2 "w_smd_trans:sot223" H 8100 8250 60  0001 C CNN
+F 2 "project:sot223" H 8100 8250 60  0001 C CNN
 F 3 "" H 8100 8250 60  0000 C CNN
 F 4 "926-M1117IMPXADJNOPB" H 8100 8300 60  0001 C CNN "Mouser Part No."
@@
 F 0 "C6" H 7400 8750 50  0000 L CNN
 F 1 "10uf/6.3V" H 7400 8550 50  0000 L CNN
-F 2 "w_smd_cap:c_elec_4x5.3" H 7450 8500 30  0001 C CNN
+F 2 "project:c_elec_4x5.3" H 7450 8500 30  0001 C CNN
 F 3 "" H 7350 8650 300 0000 C CNN
 F 4 "5985-AVS16V100-F" H 7350 8650 60  0001 C CNN "Mouser Part No."
@@
 F 0 "R8" V 8180 9300 50  0000 C CNN
 F 1 "390" V 8107 9301 50  0000 C CNN
-F 2 "w_smd_resistors:r_0402" V 8030 9300 30  0001 C CNN
+F 2 "project:r_0402" V 8030 9300 30  0001 C CNN
 F 3 "" H 8100 9300 30  0000 C CNN
 F 4 "594-MCT06030C3900FP5" V 8100 9300 60  0001 C CNN "Mouser Part No."
@@
 F 0 "R9" V 9230 8600 50  0000 C CNN
 F 1 "240" V 9157 8601 50  0000 C CNN
-F 2 "w_smd_resistors:r_0402" V 9080 8600 30  0001 C CNN
+F 2 "project:r_0402" V 9080 8600 30  0001 C CNN
 F 3 "" H 9150 8600 30  0000 C CNN
 F 4 "754-RR0816P-241D" V 9150 8600 60  0001 C CNN "Mouser Part No."
@@
 F 0 "D3" H 10550 8650 50  0000 C CNN
 F 1 "LED" H 10550 8450 50  0000 C CNN
-F 2 "w_smd_leds:Led_0603" H 10550 8550 60  0001 C CNN
+F 2 "project:Led_0603" H 10550 8550 60  0001 C CNN
 F 3 "" H 10550 8550 60  0000 C CNN
 F 4 "743-HT-191USD" H 10550 8550 60  0001 C CNN "Mouser Part No."
@@
 F 0 "R10" V 10630 9200 50  0000 C CNN
 F 1 "360" V 10557 9201 50  0000 C CNN
-F 2 "w_smd_resistors:r_0402" V 10480 9200 30  0001 C CNN
+F 2 "project:r_0402" V 10480 9200 30  0001 C CNN
 F 3 "" H 10550 9200 30  0000 C CNN
 F 4 "71-CRCW0603316RFKEB" V 10550 9200 60  0001 C CNN "Mouser Part No."
@@
 F 0 "C5" H 4800 8800 40  0000 L CNN
 F 1 "0.1uf" H 4806 8615 40  0000 L CNN
-F 2 "w_smd_cap:c_0402" H 4838 8550 30  0001 C CNN
+F 2 "project:c_0402" H 4838 8550 30  0001 C CNN
 F 3 "" H 4800 8700 60  0000 C CNN
 F 4 "810-C1005X5R1H104K" H 4800 8700 60  0001 C CNN "Mouser Part No."
@@
 F 0 "C7" H 9500 8650 40  0000 L CNN
 F 1 "0.1uf" H 9506 8465 40  0000 L CNN
-F 2 "w_smd_cap:c_0402" H 9538 8400 30  0001 C CNN
+F 2 "project:c_0402" H 9538 8400 30  0001 C CNN
 F 3 "" H 9500 8550 60  0000 C CNN
 F 4 "810-C1005X5R1H104K" H 9500 8550 60  0001 C CNN "Mouser Part No."
@@
 F 0 "P2" H 3350 7100 50  0000 C CNN
 F 1 "CONN_01X02" V 3450 6950 50  0000 C CNN
-F 2 "w_conn_mkds:mkds_1,5-2" H 3350 6950 60  0001 C CNN
+F 2 "project:mkds_1,5-2" H 3350 6950 60  0001 C CNN
 F 3 "" H 3350 6950 60  0000 C CNN
 F 4 "651-1904383" H 3350 6950 60  0001 C CNN "Mouser Part No."
@@
 F 0 "C4" H 2350 4800 40  0000 L CNN
 F 1 "0.1uf" H 2356 4615 40  0000 L CNN
-F 2 "w_smd_cap:c_0402" H 2388 4550 30  0001 C CNN
+F 2 "project:c_0402" H 2388 4550 30  0001 C CNN
 F 3 "" H 2350 4700 60  0000 C CNN
 F 4 "810-C1005X5R1H104K" H 2350 4700 60  0001 C CNN "Mouser Part No."
@@
 F 0 "C8" H 9900 8650 40  0000 L CNN
 F 1 "1uf" H 9906 8465 40  0000 L CNN
-F 2 "w_smd_cap:c_0402" H 9938 8400 30  0001 C CNN
+F 2 "project:c_0402" H 9938 8400 30  0001 C CNN
 F 3 "" H 9900 8550 60  0000 C CNN
 F 4 "810-C1005X5R1H104K" H 9900 8550 60  0001 C CNN "Mouser Part No."

Commit message: refactor large components
Parts:
- C2, C3, C4, C5, C7, C8: footprint project:c_0402 -> project:c_0805
- P3: footprint project:pin_socket_20x2 -> project:pin_socket_20x2_mirrored
- R1, R10, R2, R3, R4, R5, R6, R7, R8, R9: footprint project:r_0402 -> project:r_0805
- U2: value CAT24C32HU4I-GT3 -> CAT24C04WI-GT3; footprint project:tssop-8 -> project:CAT24C04WI-GT3; Farnell Part No. 2463727 -> 2463704; Mouser Part No. 698-CAT24C32YI-GT3 -> (none)
- U3: footprint project:sot23-6 -> project:FDC5614P
Changed lines of the file:
@@
 F 0 "P3" H 4650 5850 60  0000 C CNN
 F 1 "Raspberry_Pi_+_Conn" H 6050 2450 60  0000 C CNN
-F 2 "project:pin_socket_20x2" H 5750 3900 60  0001 C CNN
+F 2 "project:pin_socket_20x2_mirrored" H 5750 3900 60  0001 C CNN
 F 3 "" H 5750 3900 60  0000 C CNN
 F 4 "517-30340-6002" H 5750 3900 60  0001 C CNN "Mouser Part No."
@@
 P 3000 4400
 F 0 "U2" H 2900 4550 60  0000 C CNN
-F 1 "CAT24C32HU4I-GT3" H 3400 3600 60  0000 C CNN
-F 2 "project:tssop-8" H 3000 4400 60  0001 C CNN
+F 1 "CAT24C04WI-GT3" H 3150 3600 60  0000 C CNN
+F 2 "project:CAT24C04WI-GT3" H 3000 4400 60  0001 C CNN
 F 3 "" H 3000 4400 60  0000 C CNN
-F 4 "698-CAT24C32YI-GT3" H 3000 4400 60  0001 C CNN "Mouser Part No."
-F 5 "2463727" H 3000 4400 60  0001 C CNN "Farnell Part No."
+F 4 "2463704" H 3000 4400 60  0001 C CNN "Farnell Part No."
 	1    3000 4400
 	1    0    0    -1
@@
 F 0 "R1" V 2080 4650 40  0000 C CNN
 F 1 "1k" V 2007 4651 40  0000 C CNN
-F 2 "project:r_0402" V 1930 4650 30  0001 C CNN
+F 2 "project:r_0805" V 1930 4650 30  0001 C CNN
 F 3 "" H 2000 4650 30  0000 C CNN
 F 4 "754-RR0510P-102D" V 2000 4650 60  0001 C CNN "Mouser Part No."
@@
 F 0 "R3" V 3930 4000 40  0000 C CNN
 F 1 "3.9k" V 3857 4001 40  0000 C CNN
-F 2 "project:r_0402" V 3780 4000 30  0001 C CNN
+F 2 "project:r_0805" V 3780 4000 30  0001 C CNN
 F 3 "" H 3850 4000 30  0000 C CNN
 F 4 "71-CRCW04023K90FKED" V 3850 4000 60  0001 C CNN "Mouser Part No."
@@
 F 0 "R5" V 4180 4000 40  0000 C CNN
 F 1 "3.9k" V 4107 4001 40  0000 C CNN
-F 2 "project:r_0402" V 4030 4000 30  0001 C CNN
+F 2 "project:r_0805" V 4030 4000 30  0001 C CNN
 F 3 "" H 4100 4000 30  0000 C CNN
 F 4 "71-CRCW04023K90FKED" V 4100 4000 60  0001 C CNN "Mouser Part No."
@@
 F 0 "R2" V 2080 8700 40  0000 C CNN
 F 1 "24k" V 2007 8701 40  0000 C CNN
-F 2 "project:r_0402" V 1930 8700 30  0001 C CNN
+F 2 "project:r_0805" V 1930 8700 30  0001 C CNN
 F 3 "" H 2000 8700 30  0000 C CNN
 F 4 "71-CRCW0402-24K-E3" V 2000 8700 60  0001 C CNN "Mouser Part No."
@@
 F 0 "C2" H 1550 9650 40  0000 L CNN
 F 1 "0.1uf" H 1556 9465 40  0000 L CNN
-F 2 "project:c_0402" H 1588 9400 30  0001 C CNN
+F 2 "project:c_0805" H 1588 9400 30  0001 C CNN
 F 3 "" H 1550 9550 60  0000 C CNN
 F 4 "810-C1005X5R1H104K" H 1550 9550 60  0001 C CNN "Mouser Part No."
@@
 F 0 "C3" H 1800 8800 40  0000 L CNN
 F 1 "1nf" H 1806 8615 40  0000 L CNN
-F 2 "project:c_0402" H 1838 8550 30  0001 C CNN
+F 2 "project:c_0805" H 1838 8550 30  0001 C CNN
 F 3 "" H 1800 8700 60  0000 C CNN
 F 4 "810-C1005C0G2A102J5C" H 1800 8700 60  0001 C CNN "Mouser Part No."
@@
 F 0 "R4" V 3980 8700 40  0000 C CNN
 F 1 "270" V 3907 8701 40  0000 C CNN
-F 2 "project:r_0402" V 3830 8700 30  0001 C CNN
+F 2 "project:r_0805" V 3830 8700 30  0001 C CNN
 F 3 "" H 3900 8700 30  0000 C CNN
 F 4 "667-ERJ-P6WJ271V" V 3900 8700 60  0001 C CNN "Mouser Part No."
@@
 F 0 "R6" V 5130 8700 40  0000 C CNN
 F 1 "30k" V 5057 8701 40  0000 C CNN
-F 2 "project:r_0402" V 4980 8700 30  0001 C CNN
+F 2 "project:r_0805" V 4980 8700 30  0001 C CNN
 F 3 "" H 5050 8700 30  0000 C CNN
 F 4 "594-MCT06030C3002FP5" V 5050 8700 60  0001 C CNN "Mouser Part No."
@@
 F 0 "R7" V 5130 9650 40  0000 C CNN
 F 1 "10k" V 5057 9651 40  0000 C CNN
-F 2 "project:r_0402" V 4980 9650 30  0001 C CNN
+F 2 "project:r_0805" V 4980 9650 30  0001 C CNN
 F 3 "" H 5050 9650 30  0000 C CNN
 F 4 "71-CRCW0603-10K-E3" V 5050 9650 60  0001 C CNN "Mouser Part No."
@@
 F 0 "U3" H 3100 8600 60  0000 C CNN
 F 1 "FDC5614P" H 3250 8100 60  0000 C CNN
-F 2 "project:sot23-6" H 3100 8500 60  0001 C CNN
+F 2 "project:FDC5614P" H 3100 8500 60  0001 C CNN
 F 3 "" H 3100 8500 60  0000 C CNN
 F 4 "512-FDC5614P" H 3250 8350 60  0001 C CNN "Mouser Part No."
@@
 F 0 "R8" V 8180 9300 50  0000 C CNN
 F 1 "390" V 8107 9301 50  0000 C CNN
-F 2 "project:r_0402" V 8030 9300 30  0001 C CNN
+F 2 "project:r_0805" V 8030 9300 30  0001 C CNN
 F 3 "" H 8100 9300 30  0000 C CNN
 F 4 "594-MCT06030C3900FP5" V 8100 9300 60  0001 C CNN "Mouser Part No."
@@
 F 0 "R9" V 9230 8600 50  0000 C CNN
 F 1 "240" V 9157 8601 50  0000 C CNN
-F 2 "project:r_0402" V 9080 8600 30  0001 C CNN
+F 2 "project:r_0805" V 9080 8600 30  0001 C CNN
 F 3 "" H 9150 8600 30  0000 C CNN
 F 4 "754-RR0816P-241D" V 9150 8600 60  0001 C CNN "Mouser Part No."
@@
 F 0 "R10" V 10630 9200 50  0000 C CNN
 F 1 "360" V 10557 9201 50  0000 C CNN
-F 2 "project:r_0402" V 10480 9200 30  0001 C CNN
+F 2 "project:r_0805" V 10480 9200 30  0001 C CNN
 F 3 "" H 10550 9200 30  0000 C CNN
 F 4 "71-CRCW0603316RFKEB" V 10550 9200 60  0001 C CNN "Mouser Part No."
@@
 F 0 "C5" H 4800 8800 40  0000 L CNN
 F 1 "0.1uf" H 4806 8615 40  0000 L CNN
-F 2 "project:c_0402" H 4838 8550 30  0001 C CNN
+F 2 "project:c_0805" H 4838 8550 30  0001 C CNN
 F 3 "" H 4800 8700 60  0000 C CNN
 F 4 "810-C1005X5R1H104K" H 4800 8700 60  0001 C CNN "Mouser Part No."
@@
 F 0 "C7" H 9500 8650 40  0000 L CNN
 F 1 "0.1uf" H 9506 8465 40  0000 L CNN
-F 2 "project:c_0402" H 9538 8400 30  0001 C CNN
+F 2 "project:c_0805" H 9538 8400 30  0001 C CNN
 F 3 "" H 9500 8550 60  0000 C CNN
 F 4 "810-C1005X5R1H104K" H 9500 8550 60  0001 C CNN "Mouser Part No."
@@
 F 0 "C4" H 2350 4800 40  0000 L CNN
 F 1 "0.1uf" H 2356 4615 40  0000 L CNN
-F 2 "project:c_0402" H 2388 4550 30  0001 C CNN
+F 2 "project:c_0805" H 2388 4550 30  0001 C CNN
 F 3 "" H 2350 4700 60  0000 C CNN
 F 4 "810-C1005X5R1H104K" H 2350 4700 60  0001 C CNN "Mouser Part No."
@@
 F 0 "C8" H 9900 8650 40  0000 L CNN
 F 1 "1uf" H 9906 8465 40  0000 L CNN
-F 2 "project:c_0402" H 9938 8400 30  0001 C CNN
+F 2 "project:c_0805" H 9938 8400 30  0001 C CNN
 F 3 "" H 9900 8550 60  0000 C CNN
 F 4 "810-C1005X5R1H104K" H 9900 8550 60  0001 C CNN "Mouser Part No."
