File: ardas_shield/ardas_shield.sch (KiCad schematic (older format))
At the start: 28 parts, among them IC1 DS1307, P1 CONN_10, P10 CONN_01X03, P2 CONN_8, P3 CONN_8, P5 CONN_6, P6 TTL_COMM, P7 CONN_01X03, P8 CONN_01X03, P9 CONN_01X03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

Commit message: add new leds and footprints
Parts:
- removed D1: LED_RABG, kicad-gfa local:led-P-LCC-4-3, symbol LED_RABG
- added D1: LED Green, LEDs:LED_0805, symbol LED
- added D2: LED Yellow, LEDs:LED_0805, symbol LED
- added D3: LED Red, LEDs:LED_0805, symbol LED
- R2: value 4.7k -> 150 Ohm; Code_Commande (none) -> 2062238
- R3: value 10k -> 150 Ohm
- R4: value 4.7k -> 160 Ohm; Order_Code 9233881 -> 2694996
Connections:
- wire segments 193 -> 203
Changed lines of the file:
@@
 	-1   0    0    1
 $EndComp
-Text GLabel 12200 2200 0    39   Input ~ 0
-D16
 Text GLabel 11850 4800 3    39   Input ~ 0
-D17
-Text GLabel 12200 2000 0    39   Input ~ 0
 D17
 $Comp
@@
 	1    0    0    -1
 $EndComp
-$Comp
-L LED_RABG D1
-U 1 1 565885AB
-P 12800 2200
-F 0 "D1" H 12875 2550 50  0000 C CNN
-F 1 "LED_RABG" H 12825 1850 50  0000 C CNN
-F 2 "kicad-gfa local:led-P-LCC-4-3" H 12750 2150 50  0001 C CNN
-F 3 "https://github.com/UMONS-GFA/kicad-gfa.pretty/blob/master/datasheets/AV02-4186EN_DS_ASMB-MTB0_2014-09-10.pdf" H 12750 2150 50  0001 C CNN
-	1    12800 2200
-	1    0    0    -1
-$EndComp
-Text GLabel 13100 2200 2    39   Input ~ 0
-+5V
 NoConn ~ 10700 3300
-Text GLabel 12200 2400 0    39   Input ~ 0
-GND
 $Comp
 L R_PACK4 RP2
@@
 Wire Wire Line
 	6500 5800 6500 5950
-$Comp
-L R R2
-U 1 1 568BE18A
-P 12350 2000
-F 0 "R2" V 12430 2000 50  0000 C CNN
-F 1 "4.7k" V 12350 2000 50  0000 C CNN
-F 2 "kicad-gfa local:R_0805" V 12280 2000 50  0001 C CNN
-F 3 "" H 12350 2000 50  0000 C CNN
-F 4 "9233903RL " V 12350 2000 60  0001 C CNN "Order_Code"
-F 5 "YAGEO (PHYCOMP) " V 12350 2000 60  0001 C CNN "MFN"
-F 6 "RC0805JR-07150RL" V 12350 2000 60  0001 C CNN "MFP"
-F 7 "0805 [2012 Metric]" V 12350 2000 60  0001 C CNN "Case_Style"
-	1    12350 2000
-	0    1    1    0
-$EndComp
-$Comp
-L R R3
-U 1 1 568BE39C
-P 12350 2200
-F 0 "R3" V 12430 2200 50  0000 C CNN
-F 1 "10k" V 12350 2200 50  0000 C CNN
-F 2 "kicad-gfa local:R_0805" V 12280 2200 50  0001 C CNN
-F 3 "" H 12350 2200 50  0000 C CNN
-F 4 "9233881" V 12350 2200 60  0001 C CNN "Order_Code"
-F 5 "YAGEO (PHYCOMP) " V 12350 2200 60  0001 C CNN "MFN"
-F 6 "RC0805JR-07100RL" V 12350 2200 60  0001 C CNN "MFP"
-F 7 "0805 [2012 Metric]" V 12350 2200 60  0001 C CNN "Case_Style"
-	1    12350 2200
-	0    1    1    0
-$EndComp
-$Comp
-L R R4
-U 1 1 568BE4E9
-P 12350 2400
-F 0 "R4" V 12430 2400 50  0000 C CNN
-F 1 "4.7k" V 12350 2400 50  0000 C CNN
-F 2 "kicad-gfa local:R_0805" V 12280 2400 50  0001 C CNN
-F 3 "" H 12350 2400 50  0000 C CNN
-F 4 "9233881" V 12350 2400 60  0001 C CNN "Order_Code"
-F 5 "YAGEO (PHYCOMP)" V 12350 2400 60  0001 C CNN "MFN"
-F 6 "RC0805JR-07100RL" V 12350 2400 60  0001 C CNN "MFP"
-F 7 "805 [2012 Metric]" V 12350 2400 60  0001 C CNN "Case_Style"
-	1    12350 2400
-	0    1    1    0
-$EndComp
 $Comp
 L Jumper_NO_Small JP1
@@
 Text Notes 9250 6650 0    60   Italic 12
 SHOULDN'T WE SET PIN 10 TO GND OR VCC?
+$Comp
+L LED D1
+U 1 1 5B040EFB
+P 11400 1800
+F 0 "D1" H 11400 1900 50  0000 C CNN
+F 1 "LED Green" H 11400 2000 50  0000 C CNN
+F 2 "LEDs:LED_0805" H 11450 1650 50  0001 C CNN
+F 3 "" H 11400 1800 50  0000 C CNN
+F 4 "2062259" H 11400 1800 60  0001 C CNN "Order_Code"
+	1    11400 1800
+	1    0    0    -1
+$EndComp
+$Comp
+L LED D2
+U 1 1 5B040F73
+P 11400 2150
+F 0 "D2" H 11400 2250 50  0000 C CNN
+F 1 "LED Yellow" H 11400 2000 50  0000 C CNN
+F 2 "LEDs:LED_0805" H 11400 2150 50  0001 C CNN
+F 3 "" H 11400 2150 50  0000 C CNN
+F 4 "2062217" H 11400 2150 60  0001 C CNN "Order_Code"
+	1    11400 2150
+	1    0    0    -1
+$EndComp
+$Comp
+L LED D3
+U 1 1 5B040FEB
+P 11400 2500
+F 0 "D3" H 11400 2600 50  0000 C CNN
+F 1 "LED Red" H 11400 2350 50  0000 C CNN
+F 2 "LEDs:LED_0805" H 11400 2500 50  0001 C CNN
+F 3 "" H 11400 2500 50  0000 C CNN
+F 4 "2062238" H 11400 2500 60  0001 C CNN "Order_Code"
+	1    11400 2500
+	1    0    0    -1
+$EndComp
+Text GLabel 12050 2150 2    39   Input ~ 0
++5V
+Text GLabel 10750 1800 0    39   Input ~ 0
+D17
+Text GLabel 10750 2150 0    39   Input ~ 0
+D16
+Text GLabel 10750 2500 0    39   Input ~ 0
+GND
+$Comp
+L R R2
+U 1 1 5B04166A
+P 10950 1800
+F 0 "R2" V 11030 1800 50  0000 C CNN
+F 1 "150 Ohm" V 10850 1800 50  0000 C CNN
+F 2 "kicad-gfa local:R_0805" V 10880 1800 50  0001 C CNN
+F 3 "" H 10950 1800 50  0000 C CNN
+F 4 "9233903RL " V 10950 1800 60  0001 C CNN "Order_Code"
+F 5 "YAGEO (PHYCOMP) " V 10950 1800 60  0001 C CNN "MFN"
+F 6 "RC0805JR-07150RL" V 10950 1800 60  0001 C CNN "MFP"
+F 7 "0805 [2012 Metric]" V 10950 1800 60  0001 C CNN "Case_Style"
+F 8 "2062238" V 10950 1800 60  0001 C CNN "Code_Commande"
+	1    10950 1800
+	0    1    1    0
+$EndComp
+$Comp
+L R R3
+U 1 1 5B041714
+P 10950 2150
+F 0 "R3" V 11050 2150 50  0000 C CNN
+F 1 "150 Ohm" V 10850 2150 50  0000 C CNN
+F 2 "kicad-gfa local:R_0805" V 10880 2150 50  0001 C CNN
+F 3 "" H 10950 2150 50  0000 C CNN
+F 4 "9233881" V 10950 2150 60  0001 C CNN "Order_Code"
+F 5 "YAGEO (PHYCOMP) " V 10950 2150 60  0001 C CNN "MFN"
+F 6 "RC0805JR-07100RL" V 10950 2150 60  0001 C CNN "MFP"
+F 7 "0805 [2012 Metric]" V 10950 2150 60  0001 C CNN "Case_Style"
+	1    10950 2150
+	0    1    1    0
+$EndComp
+$Comp
+L R R4
+U 1 1 5B0417C3
+P 10950 2500
+F 0 "R4" V 11030 2500 50  0000 C CNN
+F 1 "160 Ohm" V 10850 2500 50  0000 C CNN
+F 2 "kicad-gfa local:R_0805" V 10880 2500 50  0001 C CNN
+F 3 "" H 10950 2500 50  0000 C CNN
+F 4 "2694996" V 10950 2500 60  0001 C CNN "Order_Code"
+F 5 "YAGEO (PHYCOMP)" V 10950 2500 60  0001 C CNN "MFN"
+F 6 "RC0805JR-07100RL" V 10950 2500 60  0001 C CNN "MFP"
+F 7 "805 [2012 Metric]" V 10950 2500 60  0001 C CNN "Case_Style"
+	1    10950 2500
+	0    1    1    0
+$EndComp
+Wire Wire Line
+	10750 2150 10800 2150
+Wire Wire Line
+	10750 1800 10800 1800
+Wire Wire Line
+	10750 2500 10800 2500
+Wire Wire Line
+	11100 1800 11200 1800
+Wire Wire Line
+	11100 2150 11200 2150
+Wire Wire Line
+	11100 2500 11200 2500
+Wire Wire Line
+	11600 1800 11800 1800
+Wire Wire Line
+	11800 1800 11800 2500
+Wire Wire Line
+	11600 2150 12050 2150
+Wire Wire Line
+	11800 2500 11600 2500
+Connection ~ 11800 2150
 $EndSCHEMATC

Commit message: replace 4 resistors groups with separated resistor 0805
Parts:
- removed RP1: R_4x4.7k, kicad-gfa local:R_Array_Convex_4x0603, symbol R_PACK4
- removed RP2, RP3, RP4, RP5: R_4x10k, kicad-gfa local:R_Array_Convex_4x0603, symbol R_PACK4
- added R10, R11, R12, R13, R14, R15, R16, R17, R18, R19, R20, R21, R22, R23, R24, R9: R_10K, Resistors_SMD:R_0805, symbol R
- added R5, R6, R7, R8: R_4.7K, Resistors_SMD:R_0805, symbol R
- U3: Supplier (none) -> Farnell
Connections:
- wire segments 203 -> 218
