File: ardas_shield/ardas_shield.sch (KiCad schematic (older format))
At the start: 45 parts, among them IC1 DS1307, P1 CONN_10, P10 CONN_01X03, P2 CONN_8, P3 CONN_8, P5 CONN_6, P6 TTL_COMM, P7 CONN_01X03, P8 CONN_01X03, P9 CONN_01X03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

Commit message: complete componenents metadatas with Kifield
Parts:
- BT1: Dealer (none) -> Farnell; Gender (none) -> 1650692; Order_Code 1650692 -> 1650692; Part Number (none) -> 1650692
- D1: Dealer (none) -> Farnell; Gender (none) -> 2062259; MFN (none) -> LUMEX; MFP (none) -> SML-LXT0805GW-TR; Part Number (none) -> 2062259
- D2: Dealer (none) -> Farnell; Gender (none) -> 2062217; MFN (none) -> LUMEX; MFP (none) -> SML-LX0805YC-TR; Part Number (none) -> 2062217
- D3: Dealer (none) -> Farnell; Gender (none) -> 2062238; MFN (none) -> LUMEX; MFP (none) -> SML-LXT0805SRW-TR; Part Number (none) -> 2062238
- IC1: Dealer (none) -> Farnell; Gender (none) -> 9725253; Part Number (none) -> 9725253
- JP1, R1: Dealer (none) -> Farnell
- P1: Dealer (none) -> Farnell; Gender (none) -> 1278412; Part Number (none) -> 1278412
- P10, P7, P8, P9: Contact_Termination_Type (none) -> Through Hole; Dealer (none) -> Farnell; MFN (none) -> MULTICOMP; MFP (none) -> MC34747; Order_Code (none) -> 1593427; Part Number (none) -> 1593427; Pitch_Spacing (none) -> 2.54mm
- P2: Contact_Termination_Type (none) -> Through Hole; Dealer (none) -> Farnell; MFN (none) -> HARWIN; MFP (none) -> M20-9990846; Order_Code (none) -> 1022257; Part Number (none) -> 1022257; Pitch_Spacing (none) -> 2.54mm
- P3: Dealer (none) -> Farnell; Gender (none) -> 1924194; MFN FCI -> HARWIN; MFP 68000-208HLF -> M20-9990846; Order_Code 1924194 -> 1022257; Part Number (none) -> 1022257
- P5: Dealer (none) -> Farnell; Gender (none) -> 2132359; Part Number (none) -> 2132359
- P6: Dealer (none) -> Farnell; Gender Header -> 1593427; Part Number (none) -> 1593427
- R10, R11, R12, R13, R14, R15, R16, R17, R18, R19, R20, R21, R22, R23, R24, R9: Case_Style (none) -> 0805 [2012 Metric]; Dealer (none) -> Farnell; MFN (none) -> MULTICOMP; MFP (none) -> MCWR08X1002FTL; Order_Code (none) -> 2447553; Part Number (none) -> 2447553
- R2: Dealer (none) -> Farnell; Gender (none) -> 2062238; Part Number (none) -> 9233903RL
- R3: Dealer (none) -> Farnell; Gender (none) -> 9233881; Part Number (none) -> 9233881
- R4: Dealer (none) -> Farnell; Gender (none) -> 2694996; Part Number (none) -> 2694996
- R5, R6, R7, R8: Case_Style (none) -> 0805 [2012 Metric]; Dealer (none) -> Farnell; MFN (none) -> YAGEO (PHYCOMP); MFP (none) -> RC0805JR-074K7L; Order_Code (none) -> 9234098; Part Number (none) -> 9234098
- U1: Case_Style (none) -> SOIC; Dealer (none) -> Farnell; Gender (none) -> 1595418; Part Number (none) -> 1595418
- U2, U4: Case_Style (none) -> SOIC; Dealer (none) -> Farnell; Gender (none) -> 9591192; Part Number (none) -> 9591192
- U3: Case_Style (none) -> TSSOP; Dealer (none) -> Farnell; Gender (none) -> 1741273; Order_Code 1741273 -> 1741273
- U6: Case_Style (none) -> TSSOP; Dealer (none) -> Farnell; Gender (none) -> 1741273; Part Number (none) -> 1741273
- X1: Case_Style (none) -> CMS, 3.2mm x 1.5mm; Dealer (none) -> Farnell; Gender (none) -> 2467865; Part Number (none) -> 2467865

Commit message: update pcbnew layout
Connections:
- net labels removed: D04
- no-connect marks 17 -> 18
