File: ardas_shield/ardas_shield.sch (KiCad schematic (older format))
At the start: 31 parts, among them IC1 DS1307, P1 CONN_10, P10 CONN_01X03, P2 CONN_8, P3 CONN_8, P4 CONN_ICSP, P5 CONN_6, P6 TTL_COMM, P7 CONN_01X03, P8 CONN_01X03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

Commit message: add values for resistors
Parts:
- R2, R3: value R -> 150 Ohm
- R4: value R -> 160 Ohm
Changed lines of the file:
@@
 P 10800 1950
 F 0 "R2" V 10880 1950 50  0000 C CNN
-F 1 "R" V 10800 1950 50  0000 C CNN
+F 1 "150 Ohm" V 10700 1950 50  0000 C CNN
 F 2 "kicad-gfa local:R_0805" V 10730 1950 50  0001 C CNN
 F 3 "" H 10800 1950 50  0000 C CNN
@@
 P 10800 2250
 F 0 "R3" V 10880 2250 50  0000 C CNN
-F 1 "R" V 10800 2250 50  0000 C CNN
+F 1 "150 Ohm" V 10700 2250 50  0000 C CNN
 F 2 "kicad-gfa local:R_0805" V 10730 2250 50  0001 C CNN
 F 3 "" H 10800 2250 50  0000 C CNN
@@
 P 10800 2550
 F 0 "R4" V 10880 2550 50  0000 C CNN
-F 1 "R" V 10800 2550 50  0000 C CNN
+F 1 "160 Ohm" V 10700 2550 50  0000 C CNN
 F 2 "kicad-gfa local:R_0805" V 10730 2550 50  0001 C CNN
 F 3 "" H 10800 2550 50  0000 C CNN
