File: ardas_shield/ardas_shield.kicad_pcb (KiCad board)
At the start: 2 copper layers, 68.6 x 53.3 mm, 49 parts, among them IC1 DS1307, P1 CONN_10, P10 CONN_01X03, P2 CONN_8, P3 CONN_8, P4 CONN_ICSP, P5 CONN_6, P6 TTL_COMM, P7 CONN_01X03, P8 CONN_01X03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

Commit message: update pcbnew layout
Parts:
- moved R8 68.9 mm to (41.7, 75.3), turned to 270 degrees
- moved R5 59.6 mm to (34.1, 95.4), turned to 270 degrees
- moved R7 56.3 mm to (68.1, 77.0), turned to 90 degrees
- moved R16 51.6 mm to (75.7, 80.4), turned to 180 degrees
- moved R6 50.9 mm to (72.5, 81.5), turned to 90 degrees
- moved R13 47.3 mm to (72.4, 85.3), turned to 90 degrees
- moved R14 45.4 mm to (62.4, 90.4), turned to 180 degrees
- moved R15 43.9 mm to (61.3, 92.7), turned to 180 degrees
- moved R21 35.2 mm to (75.5, 97.0), turned to 180 degrees
- moved R24 28.9 mm to (85.8, 103.1), turned to 270 degrees
- moved R23 28.7 mm to (83.8, 103.1), turned to 270 degrees
- moved R9 27.5 mm to (62.9, 111.3), turned to 90 degrees
- moved R12 23.4 mm to (58.4, 136.5), turned to 180 degrees
- moved R11 18.9 mm to (63.1, 136.6)
- moved R10 18.2 mm to (63.2, 131.1), turned to 180 degrees
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Routing:
- net (no net): track 209.0 -> 7.28 mm, vias 5 -> 0
- net D09: track 77.2 -> 35.5 mm, vias 1 -> 0
- net GND: track 340.8 -> 302.0 mm, vias 12 -> 9
- net D17: track 35.3 -> 6.42 mm, vias 1 -> 0
- net Net-(R5-Pad1): track 25.0 -> 0.00 mm, vias 2 -> 0
- net Net-(R22-Pad1): track 29.2 -> 5.32 mm
- net D16: track 29.7 -> 6.67 mm, vias 1 -> 0
- net Net-(R19-Pad2): track 19.4 -> 0.00 mm
- net Net-(R20-Pad2): track 17.6 -> 0.00 mm
- net Net-(R18-Pad2): track 9.93 -> 0.00 mm
- net Net-(R17-Pad2): track 8.14 -> 0.00 mm
- net Net-(R10-Pad1): track 54.2 -> 49.1 mm
- net Net-(R21-Pad2): track 6.30 -> 1.32 mm
- net +5V: track 254.0 -> 258.4 mm
- net Net-(R16-Pad1): track 34.8 -> 30.8 mm
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
Commit message: ardas_shield.rules
Parts:
- moved R5 43.6 mm to (75.8, 82.6), turned to 180 degrees
- moved R17 37.9 mm to (63.7, 101.4)
- moved R20 24.5 mm to (66.7, 118.5)
- moved R19 23.5 mm to (63.4, 118.5), turned to 180 degrees
- moved R8 6.21 mm to (40.3, 81.3), turned to 0 degrees
- turned R11 to 90 degrees
Routing:
- net Net-(R5-Pad1): track 0.00 -> 25.5 mm, vias 0 -> 2
- net Net-(R19-Pad2): track 0.00 -> 13.9 mm, vias 0 -> 2
- net Net-(R20-Pad2): track 0.00 -> 9.66 mm, vias 0 -> 2
- net Net-(R14-Pad1): track 27.7 -> 35.9 mm, vias 0 -> 2
- net (no net): track 7.28 -> 0.00 mm
- net GND: track 302.0 -> 308.6 mm
- net Net-(R15-Pad1): track 36.4 -> 40.8 mm, vias 1 -> 2
- net +5V: track 258.4 -> 261.7 mm
- net Net-(R17-Pad2): track 0.00 -> 1.57 mm, vias 0 -> 1
